File: input-filter.kicad_sch (KiCad schematic)
At the start: 20 parts

Commit message: add digikey/wuerth part numbers
* update README.md part list
Parts:
- C10, C12, C14, C29, C8: DigiKey (none) -> 399-C0603C104K3RACTUCT-ND
- D10, D3, D4, D6, D8: DigiKey (none) -> 4878-BAT54SCT-ND
- R11, R14, R15, R18, R7: DigiKey (none) -> P30KDBCT-ND
- R13, R16, R17, R19, R9: value (none) -> ~
Changed lines of the file:
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@@
 			)
 		)
+		(property "DigiKey" "399-C0603C104K3RACTUCT-ND"
+			(at 165.1 81.28 0)
+			(hide yes)
+			(show_name no)
+			(do_not_autoplace no)
+			(effects
+				(font
+					(size 1.27 1.27)
+				)
+			)
+		)
 		(pin "2"
 		)
@@
 			)
 		)
+		(property "DigiKey" "P30KDBCT-ND"
+			(at 97.79 77.47 90)
+			(hide yes)
+			(show_name no)
+			(do_not_autoplace no)
+			(effects
+				(font
+					(size 1.27 1.27)
+				)
+			)
+		)
 		(pin "2"
 		)
@@
 			)
 		)
+		(property "DigiKey" "P30KDBCT-ND"
+			(at 161.29 101.6 90)
+			(hide yes)
+			(show_name no)
+			(do_not_autoplace no)
+			(effects
+				(font
+					(size 1.27 1.27)
+				)
+			)
+		)
 		(pin "2"
 		)
@@
 			)
 		)
+		(property "DigiKey" "399-C0603C104K3RACTUCT-ND"
+			(at 101.6 106.68 0)
+			(hide yes)
+			(show_name no)
+			(do_not_autoplace no)
+			(effects
+				(font
+					(size 1.27 1.27)
+				)
+			)
+		)
 		(pin "2"
 		)
@@
 			)
 		)
+		(property "DigiKey" "4878-BAT54SCT-ND"
+			(at 125.73 83.82 0)
+			(hide yes)
+			(show_name no)
+			(do_not_autoplace no)
+			(effects
+				(font
+					(size 1.27 1.27)
+				)
+			)
+		)
 		(pin "3"
 		)
@@
 			)
 		)
-		(property "Value" ""
+		(property "Value" "~"
 			(at 113.03 107.9499 0)
 			(show_name no)
@@
 			)
 		)
+		(property "DigiKey" "399-C0603C104K3RACTUCT-ND"
+			(at 165.1 105.41 0)
+			(hide yes)
+			(show_name no)
+			(do_not_autoplace no)
+			(effects
+				(font
+					(size 1.27 1.27)
+				)
+			)
+		)
 		(pin "2"
 		)
@@
 			)
 		)
+		(property "DigiKey" "4878-BAT54SCT-ND"
+			(at 125.73 134.62 0)
+			(hide yes)
+			(show_name no)
+			(do_not_autoplace no)
+			(effects
+				(font
+					(size 1.27 1.27)
+				)
+			)
+		)
 		(pin "3"
 		)
@@
 			)
 		)
-		(property "Value" ""
+		(property "Value" "~"
 			(at 176.53 82.5499 0)
 			(show_name no)
@@
 			)
 		)
+		(property "DigiKey" "399-C0603C104K3RACTUCT-ND"
+			(at 101.6 132.08 0)
+			(hide yes)
+			(show_name no)
+			(do_not_autoplace no)
+			(effects
+				(font
+					(size 1.27 1.27)
+				)
+			)
+		)
 		(pin "2"
 		)
@@
 			)
 		)
+		(property "DigiKey" "P30KDBCT-ND"
+			(at 161.29 77.47 90)
+			(hide yes)
+			(show_name no)
+			(do_not_autoplace no)
+			(effects
+				(font
+					(size 1.27 1.27)
+				)
+			)
+		)
 		(pin "2"
 		)
@@
 			)
 		)
+		(property "DigiKey" "P30KDBCT-ND"
+			(at 97.79 128.27 90)
+			(hide yes)
+			(show_name no)
+			(do_not_autoplace no)
+			(effects
+				(font
+					(size 1.27 1.27)
+				)
+			)
+		)
 		(pin "2"
 		)
@@
 			)
 		)
+		(property "DigiKey" "399-C0603C104K3RACTUCT-ND"
+			(at 101.6 81.28 0)
+			(hide yes)
+			(show_name no)
+			(do_not_autoplace no)
+			(effects
+				(font
+					(size 1.27 1.27)
+				)
+			)
+		)
 		(pin "2"
 		)
@@
 			)
 		)
-		(property "Value" ""
+		(property "Value" "~"
 			(at 176.53 106.6799 0)
 			(show_name no)
@@
 			)
 		)
+		(property "DigiKey" "4878-BAT54SCT-ND"
+			(at 125.73 109.22 0)
+			(hide yes)
+			(show_name no)
+			(do_not_autoplace no)
+			(effects
+				(font
+					(size 1.27 1.27)
+				)
+			)
+		)
 		(pin "3"
 		)
@@
 			)
 		)
+		(property "DigiKey" "4878-BAT54SCT-ND"
+			(at 189.23 107.95 0)
+			(hide yes)
+			(show_name no)
+			(do_not_autoplace no)
+			(effects
+				(font
+					(size 1.27 1.27)
+				)
+			)
+		)
 		(pin "3"
 		)
@@
 			)
 		)
-		(property "Value" ""
+		(property "Value" "~"
 			(at 113.03 133.3499 0)
 			(show_name no)
@@
 			)
 		)
-		(property "Value" ""
+		(property "Value" "~"
 			(at 113.03 82.5499 0)
 			(show_name no)
@@
 			)
 		)
+		(property "DigiKey" "4878-BAT54SCT-ND"
+			(at 189.23 83.82 0)
+			(hide yes)
+			(show_name no)
+			(do_not_autoplace no)
+			(effects
+				(font
+					(size 1.27 1.27)
+				)
+			)
+		)
 		(pin "3"
 		)
@@
 			(at 97.79 102.87 90)
 			(hide yes)
+			(show_name no)
+			(do_not_autoplace no)
+			(effects
+				(font
+					(size 1.27 1.27)
+				)
+			)
+		)
+		(property "DigiKey" "P30KDBCT-ND"
+			(at 97.79 102.87 90)
+			(hide yes)
